Commit message: backup not working

File: linorobot2_description/urdf/controllers/diff_drive.urdf.xacro (robot description, xacro)
@@ -9,12 +9,14 @@
         <left_joint>left_wheel_joint</left_joint>
         <right_joint>right_wheel_joint</right_joint>
+        <robot_base_frame>base_footprint</robot_base_frame>
         <wheel_separation>${wheel_separation}</wheel_separation>
         <wheel_diameter>${wheel_radius * 2}</wheel_diameter>
+        !-- Limits -->
+        <!-- <max_wheel_torque>200</max_wheel_torque> -->
         <max_wheel_acceleration>1.0</max_wheel_acceleration>
-        <robot_base_frame>base_footprint</robot_base_frame>
+        <odometry_frame>odom</odometry_frame>
         <publish_odom>true</publish_odom>
-        <publish_odom_tf>false</publish_odom_tf>
+        <publish_odom_tf>true</publish_odom_tf>
         <publish_wheel_tf>true</publish_wheel_tf>
-        <odometry_frame>odom</odometry_frame>
       </plugin>
     </gazebo>

File: linorobot2_description/urdf/robots/LeoGV.urdf.xacro (robot description, xacro)
@@ -2,12 +2,13 @@
 <robot name="LeoGV" xmlns:xacro="http://ros.org/wiki/xacro">
   <xacro:include filename="$(find linorobot2_description)/urdf/2wd_properties.urdf.xacro" />
+  <!-- <xacro:include filename="$(find linorobot2_description)/urdf/inertial_macros.xacro" /> -->
   <xacro:include filename="$(find linorobot2_description)/urdf/mech/base.urdf.xacro" />
   <xacro:include filename="$(find linorobot2_description)/urdf/mech/lift_plate_LeoGV.urdf.xacro" />
   <xacro:include filename="$(find linorobot2_description)/urdf/mech/wheel.urdf.xacro" />
   <xacro:include filename="$(find linorobot2_description)/urdf/mech/caster_wheel_LeoGV.urdf.xacro" />
-  <xacro:include filename="$(find linorobot2_description)/urdf/sensors/imu.urdf.xacro" />
-  <xacro:include filename="$(find linorobot2_description)/urdf/sensors/generic_laser.urdf.xacro" />
-  <xacro:include filename="$(find linorobot2_description)/urdf/sensors/depth_sensor.urdf.xacro" />
-  <xacro:include filename="$(find linorobot2_description)/urdf/sensors/camera_LeoGV.urdf.xacro" />
+  <!-- <xacro:include filename="$(find linorobot2_description)/urdf/sensors/imu.urdf.xacro" /> -->
+  <!-- <xacro:include filename="$(find linorobot2_description)/urdf/sensors/generic_laser.urdf.xacro" /> -->
+  <!-- <xacro:include filename="$(find linorobot2_description)/urdf/sensors/depth_sensor.urdf.xacro" /> -->
+  <!-- <xacro:include filename="$(find linorobot2_description)/urdf/sensors/camera_LeoGV.urdf.xacro" /> -->
   <xacro:include filename="$(find linorobot2_description)/urdf/controllers/diff_drive.urdf.xacro" />
   <xacro:base
@@ -81,13 +82,13 @@
   </xacro:if> -->
   <!-- <xacro:imu/> -->
-  <xacro:generic_laser>
+  <!-- <xacro:generic_laser>
     <xacro:insert_block name="laser_pose" />
-  </xacro:generic_laser>
+  </xacro:generic_laser> -->
   <!-- <xacro:depth_sensor>
     <xacro:insert_block name="depth_sensor_pose" />
   </xacro:depth_sensor> -->
-  <xacro:camera_LeoGV>
+  <!-- <xacro:camera_LeoGV>
     <xacro:insert_block name="depth_sensor_pose" />
-  </xacro:camera_LeoGV>
+  </xacro:camera_LeoGV> -->
   <xacro:diff_drive_controller
     wheel_separation="${wheel_pos_y * 2}"

File: linorobot2_description/urdf/sensors/camera_LeoGV.urdf.xacro (robot description, xacro)
@@ -1,4 +1,3 @@
 <robot xmlns:xacro="http://ros.org/wiki/xacro">
-  <xacro:property name="M_PI" value="3.1415926535897931" />
   <xacro:macro name="camera_LeoGV" params="*origin">
     <!-- camera_link describes the camera at the end of the arm -->
@@ -48,5 +47,5 @@
         <child link="camera_link_optical" />
     </joint>
-    <link name="camera_link_optical"></link>
+    <!-- <link name="camera_link_optical"></link> -->
     <!-- Add a gazebo tag for the ORIGINAL camera_link (but in the plugin we reference the optical frame so that ROS can orient things correctly) -->
     <!-- Within the gazebo tag we have the sensor tag, and inside that there is (among other things) the camera tag with the camera parameters,
@@ -57,9 +56,9 @@
     <gazebo reference="camera_link">
       <sensor name="camera" type="camera">
-        <always_on>true</always_on>
+        <!-- <always_on>true</always_on> -->
         <visualize>true</visualize>
-        <update_rate>5</update_rate>
+        <update_rate>510</update_rate>
         <camera name="camera">
-          <horizontal_fov>1.50098</horizontal_fov>
+          <horizontal_fov>1.089</horizontal_fov>
           <image>
             <width>640</width>
@@ -68,15 +67,15 @@
           </image>
           <clip>
-              <near>0.02</near>
-              <far>300</far>
+              <near>0.0</near>
+              <far>8.0</far>
           </clip>
-          <noise>
+          <!-- <noise>
               <type>gaussian</type>
               <mean>0.0</mean>
               <stddev>0.007</stddev>
-          </noise>
+          </noise>           -->
         </camera>
         <plugin name="camera_controller" filename="libgazebo_ros_camera.so">
-          <ros>
+          <!-- <ros>
             <remapping>/camera/camera_info:=/camera/color/camera_info</remapping>
             <remapping>/camera/image_raw:=/camera/color/image_raw</remapping>
@@ -93,11 +92,11 @@
           <min_depth>0.015</min_depth>
           <max_depth>3.0</max_depth>
-          <hack_baseline>0.07</hack_baseline>
+          <hack_baseline>0.07</hack_baseline> -->
           <frame_name>camera_link_optical</frame_name>
-          <distortion_k1>0.00000001</distortion_k1>
+          <!-- <distortion_k1>0.00000001</distortion_k1>
           <distortion_k2>0.00000001</distortion_k2>
           <distortion_k3>0.00000001</distortion_k3>
           <distortion_t1>0.00000001</distortion_t1>
-          <distortion_t2>0.00000001</distortion_t2>
+          <distortion_t2>0.00000001</distortion_t2> -->
         </plugin>
       </sensor>

File: linorobot2_description/urdf/sensors/generic_laser.urdf.xacro (robot description, xacro)
@@ -2,5 +2,5 @@
 <robot xmlns:xacro="http://ros.org/wiki/xacro">
   <xacro:include filename="$(find linorobot2_description)/urdf/sensors/laser.urdf.xacro" />
-  <xacro:macro name="generic_laser" params="*origin">
+  <!-- <xacro:macro name="generic_laser" params="*origin">
     <xacro:laser
       update_rate="10"
@@ -29,4 +29,56 @@
       <xacro:insert_block name="origin" />
     </xacro:laser>
-  </xacro:macro>
+  </xacro:macro> -->
+  <xacro:macro name="generic_laser" params="*origin">
+    <link name="laser_frame">
+        <visual>
+            <geometry>
+                <cylinder radius="0.05" length="0.04"/>
+            </geometry>
+            <material name="red"/>
+        </visual>
+        <collision>
+            <geometry>
+                <cylinder radius="0.05" length="0.04"/>
+            </geometry>
+        </collision>
+        <xacro:inertial_cylinder mass="0.1" length="0.04" radius="0.05">
+            <origin xyz="0 0 0" rpy="0 0 0"/>
+        </xacro:inertial_cylinder>
+    </link>
+    <joint name="laser_joint" type="fixed">
+        <parent link="chassis"/>
+        <child link="laser_frame"/>
+        <!-- <origin xyz="0.1 0 0.175" rpy="0 0 0"/> -->
+        <xacro:insert_block name="origin" />
+    </joint>
+    <gazebo reference="laser_frame">
+        <material>Gazebo/Red</material>
+        <sensor name="laser" type="ray">
+            <pose> 0 0 0 0 0 0 </pose>
+            <visualize>true</visualize>
+            <update_rate>10</update_rate>
+            <ray>
+                <scan>
+                    <horizontal>
+                        <samples>360</samples>
+                        <min_angle>-3.14</min_angle>
+                        <max_angle>3.14</max_angle>
+                    </horizontal>
+                </scan>
+                <range>
+                    <min>0.3</min>
+                    <max>12</max>
+                </range>
+            </ray>
+            <plugin name="laser_controller" filename="libgazebo_ros_ray_sensor.so">
+                <ros>
+                    <argument>~/out:=scan</argument>
+                </ros>
+                <output_type>sensor_msgs/LaserScan</output_type>
+                <frame_name>laser_frame</frame_name>
+            </plugin>
+        </sensor>
+    </gazebo>
+</xacro:macro>
 </robot>
