Commit message: slam and navigation

File: linorobot2_description/urdf/2wd_properties.urdf.xacro (robot description, xacro)
@@ -24,5 +24,5 @@
   <xacro:property name="caster_wheel_y" value="0.15" />
   <xacro:property name="laser_pose">
-    <origin xyz="0.12 0 0.15" rpy="0 0 0"/>
+    <origin xyz="0.12 0 0.25" rpy="0 0 0"/>
   </xacro:property>
   <xacro:property name="depth_sensor_pose">

File: linorobot2_description/urdf/controllers/diff_drive.urdf.xacro (robot description, xacro)
@@ -17,5 +17,5 @@
         <odometry_frame>odom</odometry_frame>
         <publish_odom>true</publish_odom>
-        <publish_odom_tf>true</publish_odom_tf>
+        <publish_odom_tf>false</publish_odom_tf>
         <publish_wheel_tf>true</publish_wheel_tf>
       </plugin>

File: linorobot2_description/urdf/robots/LeoGV.urdf.xacro (robot description, xacro)
@@ -105,5 +105,4 @@
           <joint_name>left_wheel_joint</joint_name>
           <joint_name>right_wheel_joint</joint_name>
-          <joint_name>lift_plate_to_base_joint</joint_name>
       </plugin>
   </gazebo>

File: linorobot2_description/urdf/sensors/generic_laser.urdf.xacro (robot description, xacro)
@@ -36,5 +36,5 @@
         <sensor name="laser" type="ray">
             <pose> 0 0 0 0 0 0 </pose>
-            <visualize>false</visualize>
+            <visualize>true</visualize>
             <update_rate>10</update_rate>
             <ray>
