Commit message: directory naming

File: leogv_description/urdf/robots/LeoGV.urdf.xacro (robot description, xacro)
@@ -1,15 +1,15 @@
 <?xml version="1.0"?>
 <robot name="LeoGV" xmlns:xacro="http://ros.org/wiki/xacro">
-  <xacro:include filename="$(find linorobot2_description)/urdf/2wd_properties.urdf.xacro" />
-  <!-- <xacro:include filename="$(find linorobot2_description)/urdf/inertial_macros.xacro" /> -->
-  <xacro:include filename="$(find linorobot2_description)/urdf/mech/base.urdf.xacro" />
-  <xacro:include filename="$(find linorobot2_description)/urdf/mech/lift_plate_LeoGV.urdf.xacro" />
-  <xacro:include filename="$(find linorobot2_description)/urdf/mech/wheel.urdf.xacro" />
-  <xacro:include filename="$(find linorobot2_description)/urdf/mech/caster_wheel_LeoGV.urdf.xacro" />
-  <!-- <xacro:include filename="$(find linorobot2_description)/urdf/sensors/imu.urdf.xacro" /> -->
-  <xacro:include filename="$(find linorobot2_description)/urdf/sensors/generic_laser.urdf.xacro" />
-  <!-- <xacro:include filename="$(find linorobot2_description)/urdf/sensors/depth_sensor.urdf.xacro" /> -->
-  <xacro:include filename="$(find linorobot2_description)/urdf/sensors/camera_LeoGV.urdf.xacro" />
-  <xacro:include filename="$(find linorobot2_description)/urdf/controllers/diff_drive.urdf.xacro" />
+  <xacro:include filename="$(find leogv_description)/urdf/2wd_properties.urdf.xacro" />
+  <!-- <xacro:include filename="$(find leogv_description)/urdf/inertial_macros.xacro" /> -->
+  <xacro:include filename="$(find leogv_description)/urdf/mech/base.urdf.xacro" />
+  <xacro:include filename="$(find leogv_description)/urdf/mech/lift_plate_LeoGV.urdf.xacro" />
+  <xacro:include filename="$(find leogv_description)/urdf/mech/wheel.urdf.xacro" />
+  <xacro:include filename="$(find leogv_description)/urdf/mech/caster_wheel_LeoGV.urdf.xacro" />
+  <!-- <xacro:include filename="$(find leogv_description)/urdf/sensors/imu.urdf.xacro" /> -->
+  <xacro:include filename="$(find leogv_description)/urdf/sensors/generic_laser.urdf.xacro" />
+  <!-- <xacro:include filename="$(find leogv_description)/urdf/sensors/depth_sensor.urdf.xacro" /> -->
+  <xacro:include filename="$(find leogv_description)/urdf/sensors/camera_LeoGV.urdf.xacro" />
+  <xacro:include filename="$(find leogv_description)/urdf/controllers/diff_drive.urdf.xacro" />
   <xacro:base
     length="${base_length}"

File: leogv_description/urdf/sensors/generic_laser.urdf.xacro (robot description, xacro)
@@ -1,32 +1,5 @@
 <?xml version="1.0"?>
 <robot xmlns:xacro="http://ros.org/wiki/xacro">
-  <xacro:include filename="$(find linorobot2_description)/urdf/sensors/laser.urdf.xacro" />
-  <xacro:macro name="generic_laser" params="*origin">
-    <link name="laser_frame">
-        <visual>
-            <geometry>
-                <cylinder radius="0.05" length="0.04"/>
-            </geometry>
-            <material name="black"/>
-        </visual>
-        <visual>
-            <origin xyz="0 0 -0.05"/>
-            <geometry>
-                <cylinder radius="0.01" length="0.1"/>
-            </geometry>
-            <material name="black"/>
-        </visual>
-        <collision>
-            <geometry>
-                <cylinder radius="0.05" length="0.04"/>
-            </geometry>
-        </collision>
-        <!-- <xacro:inertial_cylinder mass="0.1" length="0.04" radius="0.05">
-            <origin xyz="0 0 0" rpy="0 0 0"/> -->
-        <!-- </xacro:inertial_cylinder> -->
-    </link>
-  <?xml version="1.0"?>
-<robot xmlns:xacro="http://ros.org/wiki/xacro">
-  <xacro:include filename="$(find linorobot2_description)/urdf/sensors/laser.urdf.xacro" />
+  <xacro:include filename="$(find leogv_description)/urdf/sensors/laser.urdf.xacro" />
   <xacro:macro name="generic_laser" params="*origin">
     <link name="laser_frame">
@@ -88,38 +61,3 @@
     </gazebo>
 </xacro:macro>
-</robot>  <joint name="laser_joint" type="fixed">
-        <parent link="base_link"/>
-        <child link="laser_frame"/>
-        <!-- <origin xyz="0.1 0 0.175" rpy="0 0 0"/> -->
-        <xacro:insert_block name="origin" />
-    </joint>
-    <gazebo reference="laser_frame">
-        <material>Gazebo/Black</material>
-        <sensor name="laser" type="ray">
-            <pose> 0 0 0 0 0 0 </pose>
-            <visualize>true</visualize>
-            <update_rate>10</update_rate>
-            <ray>
-                <scan>
-                    <horizontal>
-                        <samples>360</samples>
-                        <min_angle>-3.14</min_angle>
-                        <max_angle>3.14</max_angle>
-                    </horizontal>
-                </scan>
-                <range>
-                    <min>0.3</min>
-                    <max>12</max>
-                </range>
-            </ray>
-            <plugin name="laser_controller" filename="libgazebo_ros_ray_sensor.so">
-                <ros>
-                    <argument>~/out:=scan</argument>
-                </ros>
-                <output_type>sensor_msgs/LaserScan</output_type>
-                <frame_name>laser_frame</frame_name>
-            </plugin>
-        </sensor>
-    </gazebo>
-</xacro:macro>
 </robot>
