Commit message: updated dimensions

File: leogv_description/urdf/2wd_properties.urdf.xacro (robot description, xacro)
@@ -1,5 +1,5 @@
 <?xml version="1.0"?>
 <robot xmlns:xacro="http://ros.org/wiki/xacro">
-  <xacro:property name="base_length" value="0.60" />
+  <xacro:property name="base_length" value="0.62" />
   <xacro:property name="base_width" value="0.40" />
   <xacro:property name="base_height" value="0.30" />
@@ -7,6 +7,6 @@
   <xacro:property name="wheel_radius" value="0.08255" />
   <xacro:property name="wheel_width" value="0.058" />
-  <xacro:property name="wheel_pos_x" value="0.15" />
-  <xacro:property name="wheel_pos_y" value="0.25" />
+  <xacro:property name="wheel_pos_x" value="0.24" />
+  <xacro:property name="wheel_pos_y" value="0.41" />
   <xacro:property name="wheel_pos_z" value="0.08255" />
   <xacro:property name="wheel_mass" value="3" />
@@ -14,7 +14,7 @@
   <!-- <xacro:property name="front_caster_wheel" value="true" />
   <xacro:property name="rear_caster_wheel" value="true" /> -->
-  <xacro:property name="lift_plate_length" value="0.30" />
-  <xacro:property name="lift_plate_width" value="0.30" />
-  <xacro:property name="lift_plate_height" value="0.01" />
+  <xacro:property name="lift_plate_length" value="0.42" />
+  <xacro:property name="lift_plate_width" value="0.455" />
+  <xacro:property name="lift_plate_height" value="0.025" />
   <xacro:property name="lift_plate_mass" value="0.5" />
   <xacro:property name="lift_plate_wheel_pos_x" value="-0.1" />

Commit message: update dimentions

File: leogv_description/urdf/2wd_properties.urdf.xacro (robot description, xacro)
@@ -1,5 +1,5 @@
 <?xml version="1.0"?>
 <robot xmlns:xacro="http://ros.org/wiki/xacro">
-  <xacro:property name="base_length" value="0.62" />
+  <xacro:property name="base_length" value="0.60" />
   <xacro:property name="base_width" value="0.40" />
   <xacro:property name="base_height" value="0.30" />
@@ -7,6 +7,6 @@
   <xacro:property name="wheel_radius" value="0.08255" />
   <xacro:property name="wheel_width" value="0.058" />
-  <xacro:property name="wheel_pos_x" value="0.24" />
-  <xacro:property name="wheel_pos_y" value="0.41" />
+  <xacro:property name="wheel_pos_x" value="0.15" />
+  <xacro:property name="wheel_pos_y" value="0.25" />
   <xacro:property name="wheel_pos_z" value="0.08255" />
   <xacro:property name="wheel_mass" value="3" />
@@ -14,7 +14,7 @@
   <!-- <xacro:property name="front_caster_wheel" value="true" />
   <xacro:property name="rear_caster_wheel" value="true" /> -->
-  <xacro:property name="lift_plate_length" value="0.42" />
-  <xacro:property name="lift_plate_width" value="0.455" />
-  <xacro:property name="lift_plate_height" value="0.025" />
+  <xacro:property name="lift_plate_length" value="0.30" />
+  <xacro:property name="lift_plate_width" value="0.30" />
+  <xacro:property name="lift_plate_height" value="0.01" />
   <xacro:property name="lift_plate_mass" value="0.5" />
   <xacro:property name="lift_plate_wheel_pos_x" value="-0.1" />
