Commit message: update camera_leoGV.urdf.xacro

File: leogv_description/urdf/sensors/camera_LeoGV.urdf.xacro (robot description, xacro)
@@ -11,5 +11,7 @@
                 <box size="0.06 0.15 0.15" />
             </geometry>
-            <material name="white" />
+            <material name="white">
+                <color rgba="1 1 1 1"/>
+            </material>
         </visual>
         <visual>
